File: generalidades/moduladores/moduladores.kicad_pcb (KiCad board)
At the start: 2 copper layers, 21 parts, among them J2 Entradas-salidas, J3 Fuente, U5 MC1496

Commit message: Diseño final de modulador 8QAM
Parts:
- removed REF**: OSHW-Logo2_9.8x8mm_SilkScreen, Symbol:OSHW-Logo2_9.8x8mm_SilkScreen
- removed REF**: KiCad-Logo2_5mm_SilkScreen, Symbol:KiCad-Logo2_5mm_SilkScreen
- added C11: 0.1uF, Capacitor_THT:CP_Radial_D4.0mm_P1.50mm, F.Cu at (90.3, 128.2)
- added C12: 10uF, Capacitor_THT:CP_Radial_D4.0mm_P1.50mm, F.Cu at (90.3, 133.7)
- added C13: 0.1uF, Capacitor_THT:CP_Radial_D4.0mm_P1.50mm, F.Cu at (90.3, 139.3)
- added C14: 10uF, Capacitor_THT:CP_Radial_D4.0mm_P1.50mm, F.Cu at (90.3, 144.8)
- added C7: 100nF, Capacitor_THT:C_Disc_D3.0mm_W1.6mm_P2.50mm, F.Cu at (120.0, 128.0)
- added C8: 100nF, Capacitor_THT:C_Disc_D3.0mm_W1.6mm_P2.50mm, F.Cu at (143.0, 112.0)
- added Q2: 2N3904, Package_TO_SOT_THT:TO-92_Inline, F.Cu at (101.5, 142.2)
- added Q3: 2N3904, Package_TO_SOT_THT:TO-92_Inline, F.Cu at (101.5, 148.0)
- added R18: 10K, Resistor_THT:R_Axial_DIN0309_L9.0mm_D3.2mm_P12.70mm_Horizontal, F.Cu at (182.5, 92.0)
- added R19: 10K, Resistor_THT:R_Axial_DIN0309_L9.0mm_D3.2mm_P12.70mm_Horizontal, F.Cu at (167.5, 88.8)
- added R20: 1k, Resistor_THT:R_Axial_DIN0309_L9.0mm_D3.2mm_P12.70mm_Horizontal, F.Cu at (130.5, 114.0)
- added R21: 51, Resistor_THT:R_Axial_DIN0309_L9.0mm_D3.2mm_P12.70mm_Horizontal, F.Cu at (176.0, 88.0)
- added R22: 51, Resistor_THT:R_Axial_DIN0309_L9.0mm_D3.2mm_P12.70mm_Horizontal, F.Cu at (138.5, 114.0)
- added R23: 51, Resistor_THT:R_Axial_DIN0309_L9.0mm_D3.2mm_P12.70mm_Horizontal, F.Cu at (159.5, 88.7)
- added R24: 1k, Resistor_THT:R_Axial_DIN0309_L9.0mm_D3.2mm_P12.70mm_Horizontal, F.Cu at (126.2, 108.0)
- added R25: 1k, Resistor_THT:R_Axial_DIN0309_L9.0mm_D3.2mm_P12.70mm_Horizontal, F.Cu at (176.3, 101.5)
- added R26: 6.8k, Resistor_THT:R_Axial_DIN0309_L9.0mm_D3.2mm_P12.70mm_Horizontal, F.Cu at (152.0, 88.7)
- added R27: 3.9k, Resistor_THT:R_Axial_DIN0309_L9.0mm_D3.2mm_P12.70mm_Horizontal, F.Cu at (144.0, 76.0)
- added R28: 3.9k, Resistor_THT:R_Axial_DIN0309_L9.0mm_D3.2mm_P12.70mm_Horizontal, F.Cu at (155.5, 122.7)
- added R31: 100k, Resistor_THT:R_Axial_DIN0309_L9.0mm_D3.2mm_P12.70mm_Horizontal, F.Cu at (74.0, 106.6)
- added R32: 1k, Resistor_THT:R_Axial_DIN0309_L9.0mm_D3.2mm_P12.70mm_Horizontal, F.Cu at (74.0, 111.4)
- added R37: 220k, Resistor_THT:R_Axial_DIN0309_L9.0mm_D3.2mm_P12.70mm_Horizontal, F.Cu at (74.0, 116.1)
- added R38: 220k, Resistor_THT:R_Axial_DIN0309_L9.0mm_D3.2mm_P12.70mm_Horizontal, F.Cu at (74.0, 120.9)
- added R39: 220k, Resistor_THT:R_Axial_DIN0309_L9.0mm_D3.2mm_P12.70mm_Horizontal, F.Cu at (74.0, 125.6)
- added R40: 220k, Resistor_THT:R_Axial_DIN0309_L9.0mm_D3.2mm_P12.70mm_Horizontal, F.Cu at (74.0, 130.4)
- added R41: 220k, Resistor_THT:R_Axial_DIN0309_L9.0mm_D3.2mm_P12.70mm_Horizontal, F.Cu at (74.0, 135.1)
- added R42: 220k, Resistor_THT:R_Axial_DIN0309_L9.0mm_D3.2mm_P12.70mm_Horizontal, F.Cu at (74.0, 139.9)
- added RV2: 50k, Potentiometer_THT:Potentiometer_Vishay_T93YA_Vertical, F.Cu at (96.9, 135.7)
- added U4: MC1496, Package_DIP:DIP-14_W7.62mm, F.Cu at (158.5, 94.6)
- moved R30 155.1 mm to (197.5, 48.5), turned to 180 degrees
- moved R29 143.0 mm to (180.0, 39.7), turned to 90 degrees
- moved RV1 107.6 mm to (183.4, 125.5)
- moved R17 105.8 mm to (154.5, 20.5), turned to -90 degrees
- moved R9 104.3 mm to (162.5, 32.7)
- moved U5 99.7 mm to (167.0, 39.5)
- moved R10 99.6 mm to (172.3, 39.5), turned to 90 degrees
- moved R13 98.5 mm to (147.0, 55.0), turned to 180 degrees
- moved R8 88.7 mm to (154.8, 131.5), turned to 0 degrees
- moved J2 74.4 mm to (107.7, 140.5)
- moved R1 73.3 mm to (139.8, 147.5)
- moved R14 72.6 mm to (134.0, 47.5), turned to 0 degrees
- moved R12 72.2 mm to (42.2, 120.9), turned to 0 degrees
- moved R16 67.3 mm to (42.2, 139.9), turned to 0 degrees
- moved R11 50.9 mm to (42.2, 116.1), turned to 0 degrees
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Connections:
- C5 pad 1: sel_moduladora -> Bcos(wt)
- R1 pad 1: portadora -> RI(t)
- R10 pad 1: portadora -> RI(t)
- R17 pad 2: Salida -> RAI(t)
- R29 pad 1: divisor -> RI(t)
- R30 pad 1: moduladora -> I(t)
- R30 pad 2: divisor -> RI(t)
- U5 pad 1: portadora -> RI(t)
- U5 pad 6: Salida -> RAI(t)
Routing:
- net +12V: track 110.4 -> 0.00 mm
- net -12V: track 60.3 -> 0.00 mm
- net Net-(C6-Pad2): track 51.5 -> 0.00 mm
- net portadora: track 41.7 -> 0.00 mm
- net sel_moduladora: track 33.3 -> 0.00 mm
- net Net-(R1-Pad2): track 30.4 -> 0.00 mm
- net Net-(R12-Pad1): track 28.6 -> 0.00 mm
- net Salida: track 27.4 -> 0.00 mm
- net Net-(C5-Pad2): track 23.2 -> 0.00 mm
- net Net-(R12-Pad2): track 19.2 -> 0.00 mm
- net Net-(R11-Pad1): track 17.2 -> 0.00 mm
- net divisor: track 13.7 -> 0.00 mm
- net Net-(R16-Pad2): track 13.4 -> 0.00 mm
- net Net-(R8-Pad2): track 9.94 -> 0.00 mm
- net Net-(R9-Pad1): track 5.35 -> 0.00 mm
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- removed copper zone on F.Cu, net GND
Other:
- board text removed: "Divisor"
- board text removed: "Modulador balanceado"
- board text removed: "Moduladora"
- board text removed: "Portadora"
- board text removed: "Seleccionar"
- board text removed: "output"
